File: hardware/sensor-module.kicad_pcb (KiCad board)
At the start: 2 copper layers, 50 x 25 mm, 45 parts, among them J1 Atlas Schientific Conductivit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, J10 Debug UART, J2 DS18B20, J3 Huba Pressure sensor, J4 Conductivity, J5 Temperature, J6 Huba Pressure, J7 MFM Module - Left, J8 MFM Module - Right, J9 UPDI Interface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

Commit message: Hardware: add screw terminals
Parts:
- J1: footprint Connector_JST:JST_PH_S5B-PH-K_1x05_P2.00mm_Horizontal -> TerminalBlock_Phoenix:TerminalBlock_Phoenix_MPT-0,5-5-2.54_1x05_P2.54mm_Horizontal
- J2, J3: footprint Connector_JST:JST_PH_S3B-PH-K_1x03_P2.00mm_Horizontal -> TerminalBlock_Phoenix:TerminalBlock_Phoenix_MPT-0,5-3-2.54_1x03_P2.54mm_Horizontal
- J7, J8: moved to B.Cu
- moved J2 2.71 mm to (155.5, 97.0)
- moved J3 2.54 mm to (146.0, 97.0)
- moved J1 2.34 mm to (131.5, 97.0)
- turned J7 to 180 degrees
- turned J8 to 180 degrees
Routing:
- net /n3V3_ON: track 59.6 -> 43.2 mm, vias 2 -> 4
- net +3.3V_SW: track 75.8 -> 81.2 mm
- net +3.3V: track 90.1 -> 94.3 mm
- net +5V_SW: track 27.2 -> 30.4 mm
- net /TEMP_DQ: track 11.8 -> 15.0 mm
- net /EC_Rx: track 24.5 -> 27.6 mm
- net /PRES_DQ: track 11.8 -> 14.8 mm
- net /EC_Tx: track 23.6 -> 26.5 mm
- net /EC_ON: track 27.8 -> 30.2 mm
- net GND: vias 58 -> 55
