File: hardware/sensor-module.kicad_sch (KiCad schematic)
At the start: 44 parts, among them J1 Atlas Schientific Conductivit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, J10 Debug UART, J2 DS18B20, J3 Huba Pressure sensor, J4 Conductivity, J5 Temperature, J6 Huba Pressure, J7 MFM Module - Left, J8 MFM Module - Right, J9 UPDI Interface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

Commit message: Hardware: add screw terminals
Parts:
- J1: footprint Connector_JST:JST_PH_S5B-PH-K_1x05_P2.00mm_Horizontal -> TerminalBlock_Phoenix:TerminalBlock_Phoenix_MPT-0,5-5-2.54_1x05_P2.54mm_Horizontal
- J2, J3: footprint Connector_JST:JST_PH_S3B-PH-K_1x03_P2.00mm_Horizontal -> TerminalBlock_Phoenix:TerminalBlock_Phoenix_MPT-0,5-3-2.54_1x03_P2.54mm_Horizontal
